File: auto humidifier/auto humidifier.kicad_sch (KiCad schematic)
At the start: 24 parts, among them J1 5V POWER, J10 Conn_01x22, J11 Conn_01x22, J12 SERVO_LEFT_EAR, J13 SERVO_RIGHT_EAR, J2 FAN, J3 MIST, J4 SERVO HEAD, J5 DISPLAY, J6 BATTERY CHECK, J7 TEMP/HUMIDITY, J8 WATER, J9 RGB, Q1 IRLB8721, Q2 IRLB8721

Commit message: pcb1
Parts:
- removed J1: 5V POWER, symbol Connector:Screw_Terminal_01x02
- added J14: Conn_01x06, Connector_PinHeader_2.54mm:PinHeader_1x06_P2.54mm_Vertical, symbol Connector_Generic:Conn_01x06
- added J15: Conn_01x04, Connector_PinHeader_2.54mm:PinHeader_1x04_P2.54mm_Vertical, symbol Connector_Generic:Conn_01x04
- C1: footprint (none) -> Capacitor_THT:CP_Radial_D10.0mm_P5.00mm
- C2: footprint (none) -> Capacitor_SMD:C_0805_2012Metric
- J10: value Conn_01x22 -> ESP32_RIGHT; footprint (none) -> Connector_PinSocket_2.54mm:PinSocket_1x22_P2.54mm_Vertical
- J11: value Conn_01x22 -> ESP32_LEFT; footprint (none) -> Connector_PinSocket_2.54mm:PinSocket_1x22_P2.54mm_Vertical
- J12, J13, J4, J7, J9: footprint (none) -> Connector_PinHeader_2.54mm:PinHeader_1x03_P2.54mm_Vertical
- J2, J3, J8: footprint (none) -> Connector_PinHeader_2.54mm:PinHeader_1x02_P2.54mm_Vertical
- J5, J6: footprint (none) -> Connector_PinHeader_2.54mm:PinHeader_1x04_P2.54mm_Vertical
- Q1, Q2: footprint (none) -> Package_TO_SOT_THT:TO-220-3_Vertical
- R1, R2, R3, R4, R5, R6: footprint (none) -> Resistor_THT:R_Axial_DIN0204_L3.6mm_D1.6mm_P5.08mm_Vertical
Connections:
- net +5V: now also J14.1 (Pin_1), J15.3 (Pin_3)
- net GND: now also J14.2 (Pin_2), J14.6 (Pin_6), J15.2 (Pin_2), J15.4 (Pin_4)
- new net BAT+: J14.3 (Pin_3)
- new net BAT-: J14.4 (Pin_4)
- new net OUT+: J14.5 (Pin_5), J15.1 (Pin_1)
