File: auto humidifier/auto humidifier.kicad_pcb (KiCad board)
At the start: 2 copper layers, 25 parts, among them J10 ESP32_RIGHT, J11 ESP32_LEFT, J12 SERVO_LEFT_EAR, J13 SERVO_RIGHT_EAR, J14 Conn_01x06, J15 Conn_01x04, J2 FAN, J3 MIST, J4 SERVO HEAD, J5 DISPLAY, J6 BATTERY CHECK, J7 TEMP/HUMIDITY, J8 WATER, J9 RGB, Q1 IRLB8721, Q2 IRLB8721

Commit message: PCB
Parts:
- added ?: LOGO, Rocket_solder:qr_insta, F.Cu at (195.0, 60.0)
- added ?: LOGO, Rocket_solder:hackclub, F.Cu at (210.0, 75.0)
- added ?: LOGO, Rocket_solder:orph, F.Cu at (215.0, 130.0)
- moved J5 86.3 mm to (210.0, 92.5)
- moved J15 81.9 mm to (225.0, 54.9)
- moved J8 75.0 mm to (195.0, 137.5)
- moved J2 70.4 mm to (180.0, 137.5)
- moved J7 67.0 mm to (140.0, 117.5)
- moved J14 66.7 mm to (220.0, 97.4)
- moved J3 56.8 mm to (165.0, 137.5)
- moved R1 55.3 mm to (154.9, 104.2)
- moved R2 55.3 mm to (154.9, 107.4)
- moved R3 55.3 mm to (154.9, 110.5)
- moved R4 55.3 mm to (154.9, 113.7)
- moved R6 55.3 mm to (154.9, 120.0)
- moved R5 55.3 mm to (154.9, 116.8)
- moved Q1 54.5 mm to (150.0, 129.1)
- moved Q2 54.5 mm to (150.0, 135.0)
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Routing:
- net +3V3: track 0.00 -> 159.9 mm, vias 0 -> 2
- net SDA: track 0.00 -> 90.5 mm
- net SCL: track 0.00 -> 89.1 mm
- net DHT_DATA: track 0.00 -> 72.6 mm, vias 0 -> 2
- net SERVO HEAD: track 0.00 -> 68.3 mm, vias 0 -> 1
- net Net-(J9-Pin_3): track 0.00 -> 57.0 mm
- net OUT+: track 0.00 -> 55.6 mm
- net WATER_SENSOR: track 0.00 -> 53.4 mm
- net FAN_CTRL: track 0.00 -> 50.7 mm, vias 0 -> 2
- net MIST_CTRL: track 0.00 -> 47.7 mm, vias 0 -> 2
- net SERVO_RE: track 0.00 -> 41.2 mm, vias 0 -> 2
- net GND: track 0.00 -> 40.7 mm, vias 0 -> 1
- net LED_DATA: track 0.00 -> 40.3 mm, vias 0 -> 1
- net Net-(D1-A): track 0.00 -> 35.9 mm
- net Net-(J2-Pin_1): track 0.00 -> 30.9 mm
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- added copper zone on B.Cu, net +5V
- added copper zone on F.Cu, net GND
Other:
- board outline added: 99 x 99 mm
- board text added: "Automatic Humidifier by KN"
